File: test.kicad_sch (KiCad schematic)
At the start: 27 parts, among them J3 Transformer, Q2 2N4401, Q3 2N4401, Q4 2N4403, Q5 TIP30C, Q6 2N4403, Q7 2N4401, Q8 2N4403, U1 TIP29C

Commit message: changed
Parts:
- added D6: LED_I, LED_THT:LED_D5.0mm, symbol LED:CQY99
- added R5: 47k, Resistor_THT:R_Axial_DIN0207_L6.3mm_D2.5mm_P15.24mm_Horizontal, symbol Device:R
- C1, C2: footprint 860130874006 (100uF 25V Blue Cap):WCAP-ATET_8X11.5_DXL_ -> ECO-S1EP153BA (15kuF Cap):CAP_PAN_30X20_PAN
- C3, C4: footprint ECO-S1EP153BA (15kuF Cap):CAP_PAN_30X20_PAN -> 860130874006 (100uF 25V Blue Cap):WCAP-ATET_8X11.5_DXL_
Connections:
- net Earth: now also D6.2 (A); no longer C2.1, D1.2 (A), D3.2 (A), Q5.2, Q6.3 (C), R7.1
- new net: D6.1 (K), R5.2
- new net V-: C2.1, D1.2 (A), D3.2 (A), Q5.2, Q6.3 (C), R5.1, R7.1
Other:
- note added: "ASS"
- note added: "TITIES"
- moved on the sheet: C1, C2, C3, C4, D1, D2, D3, D4, D5, J3, Q2, Q3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

Commit message: test
Other:
- note added: "TITIES ass"
- note removed: "TITIES"
Changed lines of the file:
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@@
 	(generator_version "9.0")
 	(paper "A4")
-	(text "TITIES\n"
+	(text "TITIES\nass\n"
 		(exclude_from_sim no)
 		(at 50.292 52.832 0)

Commit message: test branch
Other:
- note removed: "ASS"
- note removed: "TITIES ass"
Changed lines of the file:
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@@
 	(generator_version "9.0")
 	(paper "A4")
-	(text "TITIES\nass\n"
-		(exclude_from_sim no)
-		(at 50.292 52.832 0)
-		(effects
-			(font
-				(size 1.27 1.27)
-			)
-		)
-	)
-	(text "ASS\n"
-		(exclude_from_sim no)
-		(at 51.308 48.514 0)
-		(effects
-			(font
-				(size 1.27 1.27)
-			)
-		)
-	)
 	(junction
 		(at 55.88 166.37)
