File: test.kicad_sch (KiCad schematic)
At the start: 29 parts, among them J3 Transformer, Q2 2N4401, Q3 2N4401, Q4 2N4403, Q5 TIP30C, Q6 2N4403, Q7 2N4401, Q8 2N4403, U1 TIP29C

Commit message: Updated by Bryce Wed 11/19/2025 8:55
Parts:
- added D7: 1N4004, Diode_THT:D_DO-41_SOD81_P10.16mm_Horizontal, symbol Diode:1N4004
- added Q1: 2N4401, 2N4401:TO92, symbol 2N4401:2N4401
- added R10: Fan, Resistor_THT:R_Axial_DIN0207_L6.3mm_D2.5mm_P15.24mm_Horizontal, symbol Device:R
- added R11: Parallel with power resistor, Resistor_THT:R_Axial_DIN0207_L6.3mm_D2.5mm_P15.24mm_Horizontal, symbol Device:R
- added R6: 100k, Resistor_THT:R_Axial_DIN0207_L6.3mm_D2.5mm_P15.24mm_Horizontal, symbol Device:R
- added R8: 140k, Resistor_THT:R_Axial_DIN0207_L6.3mm_D2.5mm_P15.24mm_Horizontal, symbol Device:R
- added R9: Thermoresistor, Resistor_THT:R_Axial_DIN0207_L6.3mm_D2.5mm_P15.24mm_Horizontal, symbol Device:R
- added U2: LM358_DFN, Package_DFN_QFN:DFN-8-1EP_2x2mm_P0.5mm_EP1.05x1.75mm, symbol Amplifier_Operational:LM358_DFN
Connections:
- net at Q7.2, R17.1, U1.3 (E): now also R11.1
- net at C3.2, Q7.1, R1.3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: now also R11.2
- new net: D7.1 (K), R10.1, R9.1
- new net: D7.2 (A), R6.1
- new net: Q1.1, R10.2, R8.2
- new net: Q1.3, R6.2
- new net: R8.1, R9.2

Commit message: Updated by Bryce Thu 11/20/2025 8:01
Parts:
- removed D7: 1N4004, Diode_THT:D_DO-41_SOD81_P10.16mm_Horizontal, symbol Diode:1N4004
- removed U2: LM358_DFN, Package_DFN_QFN:DFN-8-1EP_2x2mm_P0.5mm_EP1.05x1.75mm, symbol Amplifier_Operational:LM358_DFN
- added IC1: AS358AP-E1, DIP762W56P254L930H431Q8N, symbol AS358AP-E1:AS358AP-E1
- added R12: 11k, Resistor_THT:R_Axial_DIN0207_L6.3mm_D2.5mm_P15.24mm_Horizontal, symbol Device:R
- added R15: 47k, Resistor_THT:R_Axial_DIN0207_L6.3mm_D2.5mm_P15.24mm_Horizontal, symbol Device:R
- added R16: 20k, Resistor_THT:R_Axial_DIN0207_L6.3mm_D2.5mm_P15.24mm_Horizontal, symbol Device:R
- added R19: Fan, Resistor_THT:R_Axial_DIN0207_L6.3mm_D2.5mm_P15.24mm_Horizontal, symbol Device:R
- R10: value Fan -> 10k
- R6: value 100k -> 10k
- R8: value 140k -> 1k
- R9: value Thermoresistor -> thermoresistor
Connections:
- net at R10.1: now also IC1.3 (INPUT_1+), R12.2; no longer R9.1
- net at R6.1: now also R8.2, IC1.2 (INPUT_1-), R15.2
- net at Q1.2: now also R16.1
- net at R6.2: now also R10.2, IC1.1 (OUTPUT_1), R15.1, R16.2, R19.1; no longer Q1.3
- new net: IC1.4 (GND), Q1.1, R12.1, R9.1
- new net: Q1.3, R19.2

Commit message: Updated by Bryce Thu 11/20/2025 13:12
Parts:
- added C5: 100u, 860130874006 (100uF 25V Blue Cap):WCAP-ATET_8X11.5_DXL_, symbol ECO-S1EP153BA (15k uF Cap):ECOS1EP153BA
- added D7: 1N4004, Diode_THT:D_DO-41_SOD81_P10.16mm_Horizontal, symbol Diode:1N4004
- added R20: 10k, Resistor_THT:R_Axial_DIN0207_L6.3mm_D2.5mm_P15.24mm_Horizontal, symbol Device:R
Connections:
- net Earth: now also IC1.4 (GND), Q1.1, R12.1, R9.1, C5.1, R20.1
- net at IC1.1 (OUTPUT_1), R15.1, R16.2: no longer R10.2, R19.1, R6.2
- net at IC1.8 (VCC): now also R10.2, R19.1, R6.2
- net at D1.1 (K), D2.2 (A), J3.1 (Pin_1): now also D7.1 (K)
- new net: C5.2, D7.2 (A), R20.2
Other:
- moved on the sheet: R10, R12

Commit message: Updated by Bryce Thu 11/20/2025 22:02
Parts:
- removed D5, D6: LED_I, LED_THT:LED_D5.0mm, symbol LED:CQY99
- removed R2, R5: 47k, Resistor_THT:R_Axial_DIN0207_L6.3mm_D2.5mm_P15.24mm_Horizontal, symbol Device:R
- added Q9: 2N7000, Package_TO_SOT_THT:TO-92_Inline, symbol Transistor_FET:2N7000
- added SW1: SW_SPST, symbol Switch:SW_SPST
- IC1: footprint DIP762W56P254L930H431Q8N -> LIB_AS358AP-E1:DIP762W56P254L930H431Q8N
- R9: footprint Resistor_THT:R_Axial_DIN0207_L6.3mm_D2.5mm_P15.24mm_Horizontal -> Resistor_THT:R_Axial_DIN0204_L3.6mm_D1.6mm_P5.08mm_Horizontal
- renumbered C1 to Vcap+1, C2 to Vcap-1
Connections:
- net Earth: now also Vcap-1.1; no longer Vcap-1.2
- net V+: now also IC1.8 (VCC), R10.2, R19.1, R6.2; no longer Vcap+1.1
- net V-: no longer Vcap-1.1
- net Discharge: now reaches D1.1 (K), D2.2 (A), J3.1 (Pin_1)
- net Discharge: now also SW1.1 (A); no longer D7.1 (K)
- net at C5.2, D7.2 (A), R20.2: now also Q9.2 (G)
- new net: D7.1 (K), SW1.2 (B)
- new net: Q9.1 (S), Vcap+1.1
- new net: Q9.3 (D), Vcap-1.2
Other:
- moved on the sheet: C3, C4, C5, D1, D2, D3, D4, D7, IC1, J3, Q1, Q2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

Commit message: Updated by Bryce Thu 11/20/2025 22:43
Parts:
- SW1: footprint (none) -> Connector_Wire:SolderWire-0.1sqmm_1x02_P3.6mm_D0.4mm_OD1mm
Changed lines of the file:
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@@
 			)
 		)
-		(property "Footprint" ""
+		(property "Footprint" "Connector_Wire:SolderWire-0.1sqmm_1x02_P3.6mm_D0.4mm_OD1mm"
 			(at 35.56 29.21 0)
 			(effects

Commit message: Updated by Bryce Sat 11/22/2025 15:42
Parts:
- added R2: Parallel with power resistor, Resistor_THT:R_Axial_DIN0207_L6.3mm_D2.5mm_P15.24mm_Horizontal, symbol Device:R
Connections:
- net at C4.1, Q8.1 (E), R18.2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: now also R2.2
- net at Q5.3, Q8.2 (B), R18.1: now also R2.1
Changed lines of the file:
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@@
 	(wire
 		(pts
+			(xy 184.15 158.75) (xy 184.15 170.18)
+		)
+		(stroke
+			(width 0)
+			(type default)
+		)
+	)
+	(wire
+		(pts
 			(xy 158.75 6.35) (xy 158.75 36.83)
 		)
@@
 	(wire
 		(pts
+			(xy 184.15 170.18) (xy 187.96 170.18)
+		)
+		(stroke
+			(width 0)
+			(type default)
+		)
+	)
+	(wire
+		(pts
 			(xy 54.61 154.94) (xy 54.61 148.59)
 		)
@@
 	(wire
 		(pts
+			(xy 195.58 170.18) (xy 207.01 170.18)
+		)
+		(stroke
+			(width 0)
+			(type default)
+		)
+	)
+	(wire
+		(pts
 			(xy 204.47 36.83) (xy 204.47 57.15)
 		)
@@
 	(wire
 		(pts
+			(xy 207.01 158.75) (xy 207.01 170.18)
+		)
+		(stroke
+			(width 0)
+			(type default)
+		)
+	)
+	(wire
+		(pts
 			(xy 184.15 27.94) (xy 187.96 27.94)
 		)
@@
 					(unit 1)
 				)
+			)
+		)
+	)
+	(symbol
+		(lib_id "Device:R")
+		(at 191.77 170.18 90)
+		(unit 1)
+		(exclude_from_sim no)
+		(in_bom yes)
+		(on_board yes)
+		(dnp no)
+		(property "Reference" "R2"
+			(at 191.77 173.228 90)
+			(effects
+				(font
+					(size 1.27 1.27)
+				)
+			)
+		)
+		(property "Value" "Parallel with power resistor"
+			(at 191.77 175.768 90)
+			(effects
+				(font
+					(size 1.27 1.27)
+				)
+			)
+		)
+		(property "Footprint" "Resistor_THT:R_Axial_DIN0207_L6.3mm_D2.5mm_P15.24mm_Horizontal"
+			(at 191.77 171.958 90)
+			(effects
+				(font
+					(size 1.27 1.27)
+				)
+				(hide yes)
+			)
+		)
+		(property "Datasheet" "~"
+			(at 191.77 170.18 0)
+			(effects
+				(font
+					(size 1.27 1.27)
+				)
+				(hide yes)
+			)
+		)
+		(property "Description" ""
+			(at 191.77 170.18 0)
+			(effects
+				(font
+					(size 1.27 1.27)
+				)
+			)
+		)
+		(pin "2"
+		)
+		(pin "1"
+		)
+		(instances
+			(project "test"
+				(path "/bd97a8e3-4fd6-4a30-adc6-276b3ee6696b"
+					(reference "R2")
+					(unit 1)
+				)
