File: test.kicad_pcb (KiCad board)
At the start: 2 copper layers, 263.4 x 145.8 mm, 27 parts, among them J3 Transformer, Q2 2N4401, Q3 2N4401, Q4 2N4403, Q5 TIP30C, Q6 2N4403, Q7 2N4401, Q8 2N4403, U1 TIP29C

Commit message: test
Parts:
- added REF**: Reverb_BTDR-1H, Audio_Module:Reverb_BTDR-1H, F.Cu at (84.5, 88.0)

Commit message: test done
Parts:
- removed REF**: Reverb_BTDR-1H, Audio_Module:Reverb_BTDR-1H

Commit message: Updated by Bryce Thu 11/20/2025 22:43
Parts:
- removed R2: 47k, Resistor_THT:R_Axial_DIN0207_L6.3mm_D2.5mm_P15.24mm_Horizontal
- added C5: 100u, 860130874006 (100uF 25V Blue Cap):WCAP-ATET_8X11.5_DXL_, F.Cu at (164.0, 140.5)
- added D7: 1N4004, Diode_THT:D_DO-41_SOD81_P10.16mm_Horizontal, F.Cu at (168.5, 117.6)
- added H1: MountingHole, MountingHole:MountingHole_3mm, F.Cu at (299.4, 40.0)
- added H2: MountingHole, MountingHole:MountingHole_3mm, F.Cu at (388.0, 40.0)
- added H3: MountingHole, MountingHole:MountingHole_3mm, F.Cu at (388.0, 80.8)
- added H4: MountingHole, MountingHole:MountingHole_3mm, F.Cu at (299.4, 80.8)
- added H5: MountingHole, MountingHole:MountingHole_3mm, F.Cu at (300.4, 99.5)
- added H6: MountingHole, MountingHole:MountingHole_3mm, F.Cu at (389.0, 99.5)
- added H7: MountingHole, MountingHole:MountingHole_3mm, F.Cu at (300.4, 140.3)
- added H8: MountingHole, MountingHole:MountingHole_3mm, F.Cu at (389.0, 140.3)
- added IC1: AS358AP-E1, LIB_AS358AP-E1:DIP762W56P254L930H431Q8N, F.Cu at (58.1, 65.6)
- added Q1: 2N4401, 2N4401:TO92, F.Cu at (57.2, 49.4)
- added Q9: 2N7000, Package_TO_SOT_THT:TO-92_Inline, F.Cu at (163.6, 127.2)
- added R10: 10k, Resistor_THT:R_Axial_DIN0207_L6.3mm_D2.5mm_P15.24mm_Horizontal, F.Cu at (28.9, 42.1)
- added R11: Parallel with power resistor, Resistor_THT:R_Axial_DIN0207_L6.3mm_D2.5mm_P15.24mm_Horizontal, F.Cu at (248.5, 41.1)
- added R12: 11k, Resistor_THT:R_Axial_DIN0207_L6.3mm_D2.5mm_P15.24mm_Horizontal, F.Cu at (28.9, 76.0)
- added R15: 47k, Resistor_THT:R_Axial_DIN0207_L6.3mm_D2.5mm_P15.24mm_Horizontal, F.Cu at (28.9, 50.6)
- added R16: 20k, Resistor_THT:R_Axial_DIN0207_L6.3mm_D2.5mm_P15.24mm_Horizontal, F.Cu at (28.9, 59.0)
- added R19: Fan, Resistor_THT:R_Axial_DIN0207_L6.3mm_D2.5mm_P15.24mm_Horizontal, F.Cu at (28.9, 67.5)
- added R20: 10k, Resistor_THT:R_Axial_DIN0207_L6.3mm_D2.5mm_P15.24mm_Horizontal, F.Cu at (159.5, 120.1)
- added R6: 10k, Resistor_THT:R_Axial_DIN0207_L6.3mm_D2.5mm_P15.24mm_Horizontal, F.Cu at (28.9, 84.4)
- added R8: 1k, Resistor_THT:R_Axial_DIN0207_L6.3mm_D2.5mm_P15.24mm_Horizontal, F.Cu at (28.9, 92.9)
- added R9: thermoresistor, Resistor_THT:R_Axial_DIN0204_L3.6mm_D1.6mm_P5.08mm_Horizontal, F.Cu at (34.0, 101.4)
- added SW1: SW_SPST (Check Diameter), Connector_Wire:SolderWire-0.1sqmm_1x02_P3.6mm_D0.4mm_OD1mm, F.Cu at (150.5, 114.3)
- C3, C4: footprint ECO-S1EP153BA (15kuF Cap):CAP_PAN_30X20_PAN -> 860130874006 (100uF 25V Blue Cap):WCAP-ATET_8X11.5_DXL_
- Vcap+1: renamed from C1; footprint 860130874006 (100uF 25V Blue Cap):WCAP-ATET_8X11.5_DXL_ -> CAP-TH_BD25.0-P10.00-D2.3-FD(15kuF):CAP-TH_BD25.0-P10.00-D2.3-FD
- Vcap-1: renamed from C2; footprint 860130874006 (100uF 25V Blue Cap):WCAP-ATET_8X11.5_DXL_ -> CAP-TH_BD25.0-P10.00-D2.3-FD(15kuF):CAP-TH_BD25.0-P10.00-D2.3-FD
- moved C4 188.8 mm to (101.0, 37.5), turned to 0 degrees
- moved J3 144.2 mm to (173.2, 34.9), turned to 0 degrees
- moved R18 135.3 mm to (113.5, 29.9), turned to -90 degrees
- moved D1 133.2 mm to (188.0, 65.5), turned to 90 degrees
- moved D3 123.4 mm to (172.3, 65.5), turned to 90 degrees
- moved Vcap-1 117.5 mm to (195.0, 107.0)
- moved Vcap+1 116.4 mm to (195.0, 134.0)
- moved R14 113.7 mm to (123.3, 45.1)
- moved R4 107.1 mm to (121.5, 89.1), turned to 180 degrees
- moved R3 107.1 mm to (235.8, 25.9)
- moved D2 104.3 mm to (180.2, 65.5), turned to 90 degrees
- moved R7 103.1 mm to (133.0, 29.9), turned to -90 degrees
- moved Q5 102.9 mm to (108.0, 58.4), turned to -90 degrees
- moved U1 99.3 mm to (245.9, 62.9)
- moved D4 96.2 mm to (164.5, 65.5)
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Connections:
- net Net-(D1-K) renamed /Discharge
- D1 pad 2: Earth -> /V-
- D3 pad 2: Earth -> /V-
- Q5 pad 2: Earth -> /V-
- Q6 pad 3: Earth -> /V-
- R7 pad 1: Earth -> /V-
- Vcap+1 pad 1: /V+ -> Net-(Q9-S)
- Vcap-1 pad 2: Earth -> Net-(Q9-D)
Routing:
- net Earth: track 513.3 -> 0.00 mm, vias 1 -> 0
- net /V+: track 188.6 -> 0.00 mm
- net Net-(Q8-E): track 100.5 -> 0.00 mm
- net Net-(C3-Pad2): track 98.3 -> 0.00 mm
- net Net-(Q2-Pad2): track 86.8 -> 0.00 mm
- net Net-(Q4-C): track 81.2 -> 0.00 mm
- net Net-(Q3-Pad2): track 67.1 -> 0.00 mm
- net Net-(Q4-B): track 66.5 -> 0.00 mm
- net /Discharge: track 60.7 -> 0.00 mm
- net Net-(U1-E): track 52.7 -> 0.00 mm
- net Net-(D5-K): track 51.1 -> 0.00 mm
- net Net-(D3-K): track 46.8 -> 0.00 mm
- net Net-(Q8-B): track 37.9 -> 0.00 mm
- net Net-(Q6-E): track 20.8 -> 0.00 mm
- net Net-(U1-B): track 15.4 -> 0.00 mm
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Other:
- board size 263.4 x 145.8 mm -> 373.5 x 145.8 mm

Commit message: Updated by Bryce Sat 11/22/2025 15:42
Parts:
- removed H1, H2, H3, H4, H5, H6, H7, H8: MountingHole, MountingHole:MountingHole_3mm
- added R2: Parallel with power resistor, Resistor_THT:R_Axial_DIN0207_L6.3mm_D2.5mm_P15.24mm_Horizontal, F.Cu at (93.9, 139.5)
- R1, R4: value P160KN-0QC15B100K -> Potentiometer
- SW1: value SW_SPST (Check Diameter) -> SW_SPST
- moved R19 179.1 mm to (187.9, 150.0)
- moved R11 174.3 mm to (94.0, 121.8), turned to 0 degrees
- moved R10 172.9 mm to (187.9, 110.0)
- moved R15 171.9 mm to (187.9, 115.8)
- moved R16 170.9 mm to (187.9, 121.6)
- moved R9 169.6 mm to (203.5, 104.5), turned to 90 degrees
- moved R12 169.0 mm to (187.9, 133.2)
- moved R6 168.1 mm to (187.9, 139.0)
- moved R17 166.6 mm to (94.0, 117.4), turned to 0 degrees
- moved R8 162.7 mm to (187.9, 127.4)
- moved Q3 156.6 mm to (116.5, 149.9)
- moved Q2 155.4 mm to (116.5, 134.9)
- moved U1 154.8 mm to (95.4, 99.5)
- moved R3 153.7 mm to (109.1, 112.9), turned to 180 degrees
- moved Q1 150.6 mm to (179.0, 138.0), turned to 0 degrees
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Routing:
- net Earth: track 0.00 -> 285.1 mm, vias 0 -> 1
- net /V+: track 0.00 -> 202.1 mm, vias 0 -> 2
- net Net-(Q8-E): track 0.00 -> 144.9 mm, vias 0 -> 2
- net Net-(Q8-B): track 0.00 -> 122.1 mm, vias 0 -> 4
- net Net-(C3-Pad2): track 0.00 -> 116.5 mm, vias 0 -> 1
- net /Discharge: track 0.00 -> 109.8 mm, vias 0 -> 1
- net Net-(R14-Pad1): track 0.00 -> 105.2 mm, vias 0 -> 1
- net /V-: track 0.00 -> 96.1 mm, vias 0 -> 2
- net Net-(Q3-Pad2): track 0.00 -> 94.3 mm, vias 0 -> 1
- net Net-(Q4-C): track 0.00 -> 91.3 mm, vias 0 -> 2
- net Net-(D7-A): track 0.00 -> 84.4 mm
- net Net-(U1-E): track 0.00 -> 79.0 mm
- net Net-(Q6-E): track 0.00 -> 66.9 mm, vias 0 -> 1
- net Net-(R1-Pad1): track 0.00 -> 66.1 mm
- net Net-(IC1-INPUT_1+): track 0.00 -> 64.8 mm, vias 0 -> 1
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Other:
- board size 373.5 x 145.8 mm -> 116 x 57 mm
- board text added: "Transformer"
